File: layout2.kicad_pcb (KiCad board)
At the start: 2 copper layers, 68.6 x 53.3 mm, 8 parts, among them P1 Power, P2 Analog, P3 Digital, P4 Digital, P5 CONN_01X01, P6 CONN_01X01, P7 CONN_01X01, P8 CONN_01X01

Commit message: modif jg
Parts:
- added J1: Conn_01x08_Female, Capteur_AIME:RN2483_new, F.Cu at (165.6, 99.7)
- added RN2483: Lora, Capteur_AIME:RN2483_new, F.Cu at (175.4, 71.8)
- added U1: Capteur_AIME, Capteur_AIME:Capteur_AIME, F.Cu at (144.7, 101.0)
- added U2: LTC1100xN8, Package_DIP:DIP-8_W7.62mm, F.Cu at (129.9, 97.6)
Connections:
- P3 pad 1: /A5(SCL) -> Net-(P3-Pad1)
- P3 pad 2: /A4(SDA) -> Net-(P3-Pad2)
