File: layout2.sch (KiCad schematic (older format))
At the start: 20 parts, among them P1 Power, P2 Analog, P3 Digital, P4 Digital, P5 CONN_01X01, P6 CONN_01X01, P7 CONN_01X01, P8 CONN_01X01, U1 Capteur_AIME, U2 LTC1100xN8

Commit message: modif jg
Parts:
- added J1: Conn_01x08_Female, Capteur_AIME:RN2483_new, symbol Connector:Conn_01x08_Female
- RN2483: footprint (none) -> Capteur_AIME:RN2483_new
Connections:
- wire segments 84 -> 91
- no-connect marks 9 -> 10
Other:
- moved on the sheet: RN2483
Changed lines of the file:
@@
 L lora:Lora RN2483
 U 1 1 5FD9B35B
-P 7050 4600
-F 0 "RN2483" H 7158 5025 50  0000 C CNN
-F 1 "Lora" H 7158 4934 50  0000 C CNN
-F 2 "" H 7050 4600 50  0001 C CNN
-F 3 "" H 7050 4600 50  0001 C CNN
-	1    7050 4600
+P 6250 5150
+F 0 "RN2483" H 6358 5575 50  0000 C CNN
+F 1 "Lora" H 6358 5484 50  0000 C CNN
+F 2 "Capteur_AIME:RN2483_new" H 6250 5150 50  0001 C CNN
+F 3 "" H 6250 5150 50  0001 C CNN
+	1    6250 5150
 	1    0    0    -1
 $EndComp
@@
 L power:GND #PWR0104
 U 1 1 5FD9EEB6
-P 7500 4500
-F 0 "#PWR0104" H 7500 4250 50  0001 C CNN
-F 1 "GND" V 7505 4372 50  0000 R CNN
-F 2 "" H 7500 4500 50  0001 C CNN
-F 3 "" H 7500 4500 50  0001 C CNN
-	1    7500 4500
+P 6700 5050
+F 0 "#PWR0104" H 6700 4800 50  0001 C CNN
+F 1 "GND" V 6705 4922 50  0000 R CNN
+F 2 "" H 6700 5050 50  0001 C CNN
+F 3 "" H 6700 5050 50  0001 C CNN
+	1    6700 5050
 	0    -1   -1   0
 $EndComp
-Text Label 7500 4700 0    50   ~ 0
+Text Label 6700 5250 0    50   ~ 0
 1(Tx)
-Text Label 7500 4800 0    50   ~ 0
+Text Label 6700 5350 0    50   ~ 0
 0(Rx)
-Text Label 7500 4600 0    50   ~ 0
+Text Label 6700 5150 0    50   ~ 0
 2
 $Comp
 L power:+3.3V #PWR0105
 U 1 1 5FDA5336
-P 7500 4400
-F 0 "#PWR0105" H 7500 4250 50  0001 C CNN
-F 1 "+3.3V" V 7515 4528 50  0000 L CNN
-F 2 "" H 7500 4400 50  0001 C CNN
-F 3 "" H 7500 4400 50  0001 C CNN
-	1    7500 4400
+P 6700 4950
+F 0 "#PWR0105" H 6700 4800 50  0001 C CNN
+F 1 "+3.3V" V 6715 5078 50  0000 L CNN
+F 2 "" H 6700 4950 50  0001 C CNN
+F 3 "" H 6700 4950 50  0001 C CNN
+	1    6700 4950
 	0    1    1    0
 $EndComp
+$Comp
+L Connector:Conn_01x08_Female J1
+U 1 1 5FD277BF
+P 8800 4850
+F 0 "J1" H 8828 4826 50  0000 L CNN
+F 1 "Conn_01x08_Female" H 8828 4735 50  0000 L CNN
+F 2 "Capteur_AIME:RN2483_new" H 8800 4850 50  0001 C CNN
+F 3 "~" H 8800 4850 50  0001 C CNN
+	1    8800 4850
+	1    0    0    -1
+$EndComp
+$Comp
+L power:GND #PWR0106
+U 1 1 5FD2862D
+P 8600 4550
+F 0 "#PWR0106" H 8600 4300 50  0001 C CNN
+F 1 "GND" V 8605 4422 50  0000 R CNN
+F 2 "" H 8600 4550 50  0001 C CNN
+F 3 "" H 8600 4550 50  0001 C CNN
+	1    8600 4550
+	0    1    1    0
+$EndComp
+Wire Wire Line
+	8600 4650 8300 4650
+Wire Wire Line
+	8600 4750 8300 4750
+Wire Wire Line
+	8600 4850 8300 4850
+Wire Wire Line
+	8600 5050 8300 5050
+Wire Wire Line
+	8600 5150 8300 5150
+NoConn ~ 8300 5050
+Wire Wire Line
+	8600 5250 8300 5250
+Wire Wire Line
+	8600 4950 8300 4950
+$Comp
+L power:+3.3V #PWR0107
+U 1 1 5FD41EE8
+P 8300 4750
+F 0 "#PWR0107" H 8300 4600 50  0001 C CNN
+F 1 "+3.3V" V 8300 5000 50  0000 C CNN
+F 2 "" H 8300 4750 50  0000 C CNN
+F 3 "" H 8300 4750 50  0000 C CNN
+	1    8300 4750
+	0    -1   -1   0
+$EndComp
 $EndSCHEMATC
